File: BuckConverter.kicad_pcb (KiCad board)
At the start: 2 copper layers, 23.3 x 26.4 mm, 16 parts, among them U1 LT1936IMS8E

Commit message: more via's, check footprints etc.
Parts:
- added TP4: TestPoint, TestPoint:TestPoint_Loop_D2.54mm_Drill1.5mm_Beaded, F.Cu at (108.8, 62.9)
- C3: footprint Capacitor_SMD:C_0805_2012Metric_Pad1.18x1.45mm_HandSolder -> Capacitor_SMD:C_1210_3225Metric_Pad1.33x2.70mm_HandSolder
- moved J2 1.34 mm to (113.8, 78.7)
- moved R4 1.10 mm to (119.8, 74.4), turned to 180 degrees
- moved L1 0.80 mm to (111.6, 73.6)
- moved C3 0.67 mm to (115.4, 75.1)
- renumbered Vin to J1, Vout to J2, GND to TP1, Vout to TP2, Vsw to TP3
Connections:
- net Net-(D2-A) renamed /Vout
- U1 pad 9: GND -> (no net)
Routing:
- net GND: vias 74 -> 52
- removed copper zone on B.Cu, net GND
Other:
- board size 23.3 x 26.4 mm -> 23.3 x 26.8 mm
